File: CIRC/CIRC_rover_schematic/CIRC_rover_schematic.kicad_sch (KiCad schematic)
At the start: 30 parts, among them M1 Falcon500, M2 Falcon500, M3 Falcon500, M4 Falcon500, SW1 SW_SPST, SW2 SW_SPST, SW3 SW_SPST, SW4 SW_SPST, SW5 SW_SPST, SW6 SW_SPST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

Commit message: Add rst button
Parts:
- added SW8: MCU ESTOP RST, symbol Switch:SW_Push
Connections:
- net at DCDC1.1 (VIN+), SW2.2 (B): now also SW8.2
- net BATT+: now reaches BT1.1 (+), BT2.1 (+), LEV200A5NAA?.2 (A2), LEV200A5NAA?.3 (+)
- net BATT+: now also SW8.1
Changed lines of the file:
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@@
 		)
 	)
-	(text_box "Network"
+	(text_box "Network\nSTM32"
 		(exclude_from_sim no)
 		(at 304.8 52.07 0)
@@
 	)
 	(junction
+		(at 233.68 53.34)
+		(diameter 0)
+		(color 255 0 0 1)
+	)
+	(junction
 		(at 261.62 39.37)
 		(diameter 0)
@@
 	(wire
 		(pts
+			(xy 210.82 53.34) (xy 218.44 53.34)
+		)
+		(stroke
+			(width 0)
+			(type default)
+		)
+	)
+	(wire
+		(pts
 			(xy 166.37 180.34) (xy 173.99 180.34)
 		)
@@
 	(wire
 		(pts
+			(xy 228.6 53.34) (xy 233.68 53.34)
+		)
+		(stroke
+			(width 0)
+			(type default)
+		)
+	)
+	(wire
+		(pts
 			(xy 233.68 53.34) (xy 270.51 53.34)
 		)
@@
 		)
 	)
+	(label "BATT+"
+		(at 210.82 53.34 0)
+		(effects
+			(font
+				(size 1.27 1.27)
+			)
+			(justify left bottom)
+		)
+	)
 	(label "X2"
 		(at 93.98 218.44 0)
@@
 		)
 	)
+	(label "BATT+"
+		(at 142.24 160.02 90)
+		(effects
+			(font
+				(size 1.27 1.27)
+			)
+			(justify left bottom)
+		)
+	)
 	(symbol
 		(lib_id "Device:LED")
@@
 					(unit 1)
 				)
+			)
+		)
+	)
+	(symbol
+		(lib_id "Switch:SW_Push")
+		(at 223.52 53.34 0)
+		(unit 1)
+		(exclude_from_sim no)
+		(in_bom yes)
+		(on_board yes)
+		(dnp no)
+		(fields_autoplaced yes)
+		(property "Reference" "SW8"
+			(at 223.52 45.72 0)
+			(effects
+				(font
+					(size 1.27 1.27)
+				)
+				(hide yes)
+			)
+		)
+		(property "Value" "MCU ESTOP RST"
+			(at 223.52 48.26 0)
+			(effects
+				(font
+					(size 1.27 1.27)
+				)
+			)
+		)
+		(property "Footprint" ""
+			(at 223.52 48.26 0)
+			(effects
+				(font
+					(size 1.27 1.27)
+				)
+				(hide yes)
+			)
+		)
+		(property "Datasheet" "~"
+			(at 223.52 48.26 0)
+			(effects
+				(font
+					(size 1.27 1.27)
+				)
+				(hide yes)
+			)
+		)
+		(property "Description" "Push button switch, generic, two pins"
+			(at 223.52 53.34 0)
+			(effects
+				(font
+					(size 1.27 1.27)
+				)
+				(hide yes)
+			)
+		)
+		(pin "1"
+		)
+		(pin "2"
+		)
+		(instances
+			(project ""
+				(path "/d297f264-241d-43d6-8daf-4cac4e29df98"
+					(reference "SW8")
+					(unit 1)
+				)

Commit message: adding bus amps
Connections:
- net GND BUS (180A): now reaches ARM1.2 (-), DCDC1.2 (VIN-), DCDC2.2 (VIN-), DCDC3.2 (VIN-), DCDC4.2 (VIN-), F6.2, LED2.1 (K), M1.1 (-), M2.1 (-), M3.1 (-), M4.1 (-), SW7.2 (B)
Other:
- note added: "160A"
- note added: "180A"
- note added: "500A Contact Rating 40 ohms Coil Resistance"
- note added: "ARM 40A expected max current"
- note added: "Brushless Motors 30A expected max current"
Changed lines of the file:
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@@
 		(comment 1 "Coco Lu")
+	)
+	(text "180A"
+		(exclude_from_sim no)
+		(at 149.352 128.778 0)
+		(effects
+			(font
+				(size 1.27 1.27)
+			)
+		)
+	)
+	(text "160A"
+		(exclude_from_sim no)
+		(at 142.494 81.788 0)
+		(effects
+			(font
+				(size 1.27 1.27)
+			)
+		)
+	)
+	(text "500A Contact Rating\n40 ohms Coil Resistance"
+		(exclude_from_sim no)
+		(at 112.776 137.922 0)
+		(effects
+			(font
+				(size 1.27 1.27)
+			)
+		)
+	)
+	(text "ARM\n40A expected \nmax current"
+		(exclude_from_sim no)
+		(at 133.604 64.262 0)
+		(effects
+			(font
+				(size 1.27 1.27)
+			)
+		)
+	)
+	(text "Brushless Motors\n30A expected max \ncurrent"
+		(exclude_from_sim no)
+		(at 60.96 51.562 0)
+		(effects
+			(font
+				(size 1.27 1.27)
+			)
+		)
 	)
 	(text_box "TPLink\nJetson (2.5A max)"
@@
 		)
 	)
-	(text_box "ESTOP CIRCUIT"
+	(text_box "ESTOP CIRCUIT (UNDER 2A)"
 		(exclude_from_sim no)
 		(at 78.74 205.74 0)
@@
 		)
 	)
+	(label "GND BUS (180A)"
+		(at 173.99 39.37 0)
+		(effects
+			(font
+				(size 1.27 1.27)
+			)
+			(justify left bottom)
+		)
+	)
